File: ESP32-Ethgate.kicad_sch (KiCad schematic)
At the start: 56 parts, among them J1 USB_B_Micro, J2 HR911105A, J3 USB, J4 GPIO, Q1 UMH3N, U1 HT7233, U2 ESP32-WROOM-32U, U3 CH340C, U4 HT7233, U5 LAN8720A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

Commit message: update the various extra files
Other:
- moved on the sheet: R23
Changed lines of the file:
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@@
     (stroke (width 0) (type default) (color 0 0 0 0))
   )
-  (wire (pts (xy 151.13 175.26) (xy 149.86 175.26))
+  (wire (pts (xy 144.78 181.61) (xy 143.51 181.61))
     (stroke (width 0) (type default) (color 0 0 0 0))
   )
@@
     (stroke (width 0) (type default) (color 0 0 0 0))
   )
-  (wire (pts (xy 156.21 175.26) (xy 156.21 179.07))
+  (wire (pts (xy 149.86 181.61) (xy 149.86 185.42))
     (stroke (width 0) (type default) (color 0 0 0 0))
   )
@@
     (stroke (width 0) (type default) (color 0 0 0 0))
   )
-  (wire (pts (xy 149.86 175.26) (xy 149.86 179.07))
+  (wire (pts (xy 143.51 181.61) (xy 143.51 185.42))
     (stroke (width 0) (type default) (color 0 0 0 0))
   )
@@
     (pin "1")
   )
-  (symbol (lib_id "Device:R_Small") (at 153.67 175.26 270) (unit 1)
-    (in_bom yes) (on_board yes)
-    (property "Reference" "R23" (id 0) (at 153.67 170.2816 90))
-    (property "Value" "0R" (id 1) (at 153.67 172.593 90))
-    (property "Footprint" "Resistor_SMD:R_0603_1608Metric" (id 2) (at 153.67 175.26 0)
-      (effects (font (size 1.27 1.27)) hide)
-    )
-    (property "Datasheet" "~" (id 3) (at 153.67 175.26 0)
+  (symbol (lib_id "Device:R_Small") (at 147.32 181.61 270) (unit 1)
+    (in_bom yes) (on_board yes)
+    (property "Reference" "R23" (id 0) (at 147.32 176.6316 90))
+    (property "Value" "0R" (id 1) (at 147.32 178.943 90))
+    (property "Footprint" "Resistor_SMD:R_0603_1608Metric" (id 2) (at 147.32 181.61 0)
+      (effects (font (size 1.27 1.27)) hide)
+    )
+    (property "Datasheet" "~" (id 3) (at 147.32 181.61 0)
       (effects (font (size 1.27 1.27)) hide)
     )
@@
     (pin "SH")
   )
-  (symbol (lib_id "power:GND") (at 149.86 179.07 0) (unit 1)
-    (in_bom yes) (on_board yes)
-    (property "Reference" "#PWR0118" (id 0) (at 149.86 185.42 0)
-      (effects (font (size 1.27 1.27)) hide)
-    )
-    (property "Value" "GND" (id 1) (at 149.987 183.4642 0))
-    (property "Footprint" "" (id 2) (at 149.86 179.07 0)
-      (effects (font (size 1.27 1.27)) hide)
-    )
-    (property "Datasheet" "" (id 3) (at 149.86 179.07 0)
-      (effects (font (size 1.27 1.27)) hide)
-    )
-    (pin "1")
-  )
-  (symbol (lib_id "power:GND1") (at 156.21 179.07 0) (unit 1)
-    (in_bom yes) (on_board yes)
-    (property "Reference" "#PWR0119" (id 0) (at 156.21 185.42 0)
-      (effects (font (size 1.27 1.27)) hide)
-    )
-    (property "Value" "GND1" (id 1) (at 156.337 183.4642 0))
-    (property "Footprint" "" (id 2) (at 156.21 179.07 0)
-      (effects (font (size 1.27 1.27)) hide)
-    )
-    (property "Datasheet" "" (id 3) (at 156.21 179.07 0)
-      (effects (font (size 1.27 1.27)) hide)
-    )
+  (symbol (lib_id "power:GND") (at 143.51 185.42 0) (unit 1)
+    (in_bom yes) (on_board yes)
+    (property "Reference" "#PWR0118" (id 0) (at 143.51 191.77 0)
+      (effects (font (size 1.27 1.27)) hide)
+    )
+    (property "Value" "GND" (id 1) (at 143.637 189.8142 0))
+    (property "Footprint" "" (id 2) (at 143.51 185.42 0)
+      (effects (font (size 1.27 1.27)) hide)
+    )
+    (property "Datasheet" "" (id 3) (at 143.51 185.42 0)
+      (effects (font (size 1.27 1.27)) hide)
+    )
+    (pin "1")
+  )
+  (symbol (lib_id "power:GND1") (at 149.86 185.42 0) (unit 1)
+    (in_bom yes) (on_board yes)
+    (property "Reference" "#PWR0119" (id 0) (at 149.86 191.77 0)
+      (effects (font (size 1.27 1.27)) hide)
+    )
+    (property "Value" "GND1" (id 1) (at 149.987 189.8142 0))
+    (property "Footprint" "" (id 2) (at 149.86 185.42 0)
+      (effects (font (size 1.27 1.27)) hide)
+    )
+    (property "Datasheet" "" (id 3) (at 149.86 185.42 0)
+      (effects (font (size 1.27 1.27)) hide)
+    )

Commit message: properly fix the nINTSEL for #1 (and document the bootstrap settings in the schematic so I remember next time).
this implicitly updates to Kicad 7.
Connections:
- net +3.3VA: now also J2.9
- net GND1: no longer J2.10
- net LINKLED: now also R17.2; no longer R17.1
- new net: J2.10, R17.1
Other:
- note added: "LAN8720A Bootstrap pins: PHYAD0 = 1 MODE[2:0] = 111 (MCU needs to pull MODE[01] high) REGOFF = 0 = enable 1.2V internal regulator nINTSEL = 1 = external clock"
- moved on the sheet: R17
