File: ESP32-Ethgate.kicad_pcb (KiCad board)
At the start: 2 copper layers, 71.2 x 38.1 mm, 56 parts, among them J1 USB_B_Micro, J2 HR911105A, J3 USB, J4 GPIO, Q1 UMH3N, U1 HT7233, U2 ESP32-WROOM-32U, U3 CH340C, U4 HT7233, U5 LAN8720A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

Commit message: small tweaks
Routing:
- net +3.3VA: track 94.0 -> 95.0 mm
Changed lines of the file:
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@@
   (via (at 90.297 83.5152) (size 1.2) (drill 0.6) (layers "F.Cu" "B.Cu") (net 4))
   (via (at 90.424 97.282) (size 1.2) (drill 0.6) (layers "F.Cu" "B.Cu") (net 4))
+  (segment (start 70.782 81.635) (end 71.6868 81.635) (width 0.4) (layer "B.Cu") (net 4))
+  (segment (start 71.6868 81.635) (end 73.112 83.0602) (width 0.4) (layer "B.Cu") (net 4))
   (segment (start 90.297 83.5152) (end 89.027 83.5152) (width 0.4) (layer "B.Cu") (net 4))
   (segment (start 80.0862 88.9) (end 82.042 88.9) (width 0.4) (layer "B.Cu") (net 4))
+  (segment (start 73.112 83.0602) (end 73.112 84.0002) (width 0.4) (layer "B.Cu") (net 4))
   (segment (start 90.3986 92.2274) (end 90.424 92.2528) (width 0.4) (layer "B.Cu") (net 4))
   (segment (start 90.424 92.2528) (end 90.424 97.282) (width 0.4) (layer "B.Cu") (net 4))
   (segment (start 79.502 85.5726) (end 79.502 88.3158) (width 0.4) (layer "B.Cu") (net 4))
-  (segment (start 71.6868 81.635) (end 74.757 84.7052) (width 0.4) (layer "B.Cu") (net 4))
   (segment (start 89.0778 88.1126) (end 88.5698 87.6046) (width 0.4) (layer "B.Cu") (net 4))
   (segment (start 89.0778 88.138) (end 89.0778 88.1126) (width 0.4) (layer "B.Cu") (net 4))
   (segment (start 90.424 88.5444) (end 90.2716 88.392) (width 0.4) (layer "B.Cu") (net 4))
-  (segment (start 70.782 81.635) (end 71.6868 81.635) (width 0.4) (layer "B.Cu") (net 4))
   (segment (start 88.5698 87.6046) (end 84.5974 87.6046) (width 0.4) (layer "B.Cu") (net 4))
+  (segment (start 74.157 85.0452) (end 79.502 85.0452) (width 0.4) (layer "B.Cu") (net 4))
   (segment (start 79.502 88.3158) (end 80.0862 88.9) (width 0.4) (layer "B.Cu") (net 4))
   (segment (start 79.502 83.2866) (end 79.502 84.7052) (width 0.4) (layer "B.Cu") (net 4))
   (segment (start 90.3732 83.5914) (end 90.3732 88.2904) (width 0.4) (layer "B.Cu") (net 4))
+  (segment (start 73.112 84.0002) (end 74.157 85.0452) (width 0.4) (layer "B.Cu") (net 4))
   (segment (start 90.2716 88.392) (end 89.3318 88.392) (width 0.4) (layer "B.Cu") (net 4))
-  (segment (start 74.757 84.7052) (end 79.502 84.7052) (width 0.4) (layer "B.Cu") (net 4))
   (segment (start 87.7062 82.1944) (end 80.5942 82.1944) (width 0.4) (layer "B.Cu") (net 4))
   (segment (start 90.3986 92.2274) (end 90.424 92.202) (width 0.4) (layer "B.Cu") (net 4))
@@
   (segment (start 90.3732 88.2904) (end 90.2716 88.392) (width 0.4) (layer "B.Cu") (net 4))
   (segment (start 90.424 92.202) (end 90.424 88.5444) (width 0.4) (layer "B.Cu") (net 4))
+  (segment (start 79.502 85.0452) (end 79.502 84.7052) (width 0.4) (layer "B.Cu") (net 4))
   (segment (start 89.3318 88.392) (end 89.0778 88.138) (width 0.4) (layer "B.Cu") (net 4))
   (segment (start 80.5942 82.1944) (end 79.502 83.2866) (width 0.4) (layer "B.Cu") (net 4))
